File: pcb/BananaGuard.kicad_pcb (KiCad board)
At the start: 2 copper layers, 49.1 x 106.6 mm, 15 parts, among them J1 AudioJack3_Ground, J2 AudioJack3_Ground, P1 USB_C_Plug_USB2.0, U1 TLV320AIC32IRHBR, U2 STM32F429VITx

Commit message: 🎛  wip analogue front end
Parts:
- added C1: 100n, Capacitor_SMD:C_0603_1608Metric, B.Cu at (133.5, 79.5)
- added C10: 100n, Capacitor_SMD:C_0603_1608Metric, B.Cu at (137.5, 79.5)
- added C11: 10u, Capacitor_SMD:CP_Elec_4x3, B.Cu at (142.5, 77.7)
- added C12: 100n, Capacitor_SMD:C_0603_1608Metric, B.Cu at (137.5, 82.0)
- added C13: 20p, Capacitor_SMD:C_0603_1608Metric, B.Cu at (137.5, 84.5)
- added C14: 2.2u, Capacitor_SMD:C_0603_1608Metric, B.Cu at (128.0, 108.0)
- added C15: 2.2u, Capacitor_SMD:C_0603_1608Metric, B.Cu at (129.2, 109.3)
- added C16: 1u, Capacitor_SMD:CP_Elec_4x3, B.Cu at (142.5, 83.5)
- added C17: 100n, Capacitor_SMD:C_0603_1608Metric, B.Cu at (137.5, 87.0)
- added C18: 1u, Capacitor_SMD:CP_Elec_4x3, B.Cu at (142.5, 89.3)
- added C19: 0.1u, Capacitor_SMD:C_0603_1608Metric, B.Cu at (125.4, 122.3)
- added C2: 10n, Capacitor_SMD:C_0603_1608Metric, B.Cu at (133.5, 82.0)
- added C20: 1u, Capacitor_SMD:CP_Elec_4x3, B.Cu at (119.5, 124.0)
- added C21: 0.1u, Capacitor_SMD:C_0603_1608Metric, B.Cu at (125.4, 124.8)
- added C22: 1u, Capacitor_SMD:CP_Elec_4x3, B.Cu at (119.5, 129.8)
- added C23: 0.1u, Capacitor_SMD:C_0603_1608Metric, B.Cu at (125.4, 127.3)
- added C24: 1u, Capacitor_SMD:CP_Elec_4x3, B.Cu at (130.7, 117.1)
- added C25: 0.1u, Capacitor_SMD:C_0603_1608Metric, B.Cu at (125.4, 129.9)
- added C26: 1u, Capacitor_SMD:CP_Elec_4x3, B.Cu at (130.7, 123.0)
- added C27: 10u, Capacitor_SMD:CP_Elec_4x3, B.Cu at (130.7, 128.8)
- added C28: 0.1u, Capacitor_SMD:C_0603_1608Metric, B.Cu at (125.4, 132.4)
- added C29: 1u, Capacitor_SMD:CP_Elec_4x3, B.Cu at (130.7, 134.7)
- added C3: 100n, Capacitor_SMD:C_0603_1608Metric, B.Cu at (133.5, 84.5)
- added C4: 10u, Capacitor_SMD:CP_Elec_4x3, B.Cu at (131.5, 56.0)
- added C5: 100n, Capacitor_SMD:C_0603_1608Metric, B.Cu at (133.5, 87.0)
- added C6: 100n, Capacitor_SMD:C_0603_1608Metric, B.Cu at (133.5, 89.5)
- added C7: 10u, Capacitor_SMD:CP_Elec_4x3, B.Cu at (128.2, 68.0)
- added C8: 100n, Capacitor_SMD:C_0603_1608Metric, B.Cu at (135.8, 91.5)
- added C9: 20p, Capacitor_SMD:C_0603_1608Metric, B.Cu at (145.0, 94.0)
- added D5: WS2812, LED_SMD:LED_WS2812_PLCC6_5.0x5.0mm_P1.6mm, F.Cu at (166.1, 49.6)
- added D6: LED, LED_SMD:LED_0603_1608Metric_Pad1.05x0.95mm_HandSolder, B.Cu at (125.5, 93.3)
- added D7: LED, LED_SMD:LED_0603_1608Metric_Pad1.05x0.95mm_HandSolder, B.Cu at (127.3, 91.5)
- added FB1: 120R, Resistor_SMD:R_0603_1608Metric, B.Cu at (137.5, 89.5)
- added J3: Conn_01x04_Pin, Connector_PinHeader_2.54mm:PinHeader_1x04_P2.54mm_Vertical, B.Cu at (135.8, 138.0)
- added J4: Conn_01x04_Pin, Connector_PinHeader_2.54mm:PinHeader_1x04_P2.54mm_Vertical, B.Cu at (120.9, 144.5)
- added J5: Conn_01x04_Pin, Connector_PinHeader_2.54mm:PinHeader_1x04_P2.54mm_Vertical, B.Cu at (151.5, 136.5)
- added R10: 270, Resistor_SMD:R_0603_1608Metric_Pad0.98x0.95mm_HandSolder, B.Cu at (130.3, 94.6)
- added R11: 270, Resistor_SMD:R_0603_1608Metric_Pad0.98x0.95mm_HandSolder, B.Cu at (132.1, 92.9)
- added R5: 1k, Resistor_SMD:R_0603_1608Metric_Pad0.98x0.95mm_HandSolder, B.Cu at (147.9, 84.0)
- added R6: 0, Resistor_SMD:R_0603_1608Metric_Pad0.98x0.95mm_HandSolder, B.Cu at (147.9, 86.5)
- added R7: 0, Resistor_SMD:R_0603_1608Metric_Pad0.98x0.95mm_HandSolder, B.Cu at (147.9, 89.0)
- added R8: 1k, Resistor_SMD:R_0603_1608Metric_Pad0.98x0.95mm_HandSolder, B.Cu at (136.8, 126.2)
- added R9: 1k, Resistor_SMD:R_0603_1608Metric_Pad0.98x0.95mm_HandSolder, B.Cu at (136.8, 128.7)
- added RV1: 10k, Potentiometer_THT:Potentiometer_Bourns_PTV09A-1_Single_Vertical, F.Cu at (156.5, 88.5)
- added RV2: 10k, Potentiometer_THT:Potentiometer_Bourns_PTV09A-1_Single_Vertical, F.Cu at (156.4, 102.3)
- added RV3: 10k, Potentiometer_THT:Potentiometer_Bourns_PTV09A-1_Single_Vertical, F.Cu at (156.4, 116.2)
- added RV4: 10k, Potentiometer_THT:Potentiometer_Bourns_PTV09A-1_Single_Vertical, F.Cu at (156.4, 130.0)
- added SW1: SW_Push, Button_Switch_SMD:Panasonic_EVQPUK_EVQPUB, B.Cu at (120.5, 75.0)
- added SW2: SW_Push_SPDT, Button_Switch_SMD:SW_SPDT_PCM12, B.Cu at (120.5, 83.5)
- added U3: NCP1117-3.3_SOT223, Package_TO_SOT_SMD:SOT-223-3_TabPin2, B.Cu at (130.0, 62.0)
- added Y1: 25 MHz, Crystal:Crystal_SMD_2520-4Pin_2.5x2.0mm, B.Cu at (147.0, 96.0)
- D4, R1, R2, R3, R4: moved to B.Cu
- moved R4 59.3 mm to (128.5, 96.4), turned to -45 degrees
- moved R1 43.6 mm to (139.0, 55.0), turned to 180 degrees
- moved R2 43.6 mm to (139.0, 57.5), turned to 180 degrees
- moved R3 43.6 mm to (139.0, 60.0), turned to 180 degrees
- moved D4 33.9 mm to (129.1, 89.6), turned to 135 degrees
- moved D1 21.7 mm to (144.5, 47.4)
- moved J1 16.8 mm to (155.5, 157.8)
- moved D2 16.6 mm to (141.3, 43.9)
- moved J2 14.8 mm to (126.5, 155.0)
- moved D3 13.4 mm to (134.2, 45.9)
- moved H1 11.3 mm to (141.0, 157.5)
- moved P1 9.76 mm to (120.5, 59.5), turned to 75 degrees
- moved H2 4.65 mm to (138.5, 73.0)
- moved U1 0.20 mm to (139.5, 120.0)
Connections:
- D4 pad 1: unconnected-(D4-K-Pad1) -> GND
- D4 pad 2: unconnected-(D4-A-Pad2) -> Net-(D4-A)
- P1 pad A4: +5V -> VBUS
- P1 pad A6: unconnected-(P1-D+-PadA6) -> /USB_D+
- P1 pad A7: unconnected-(P1-D--PadA7) -> /USB_D-
- P1 pad A9: +5V -> VBUS
- P1 pad B4: +5V -> VBUS
- P1 pad B9: +5V -> VBUS
- R1 pad 1: +5V -> /HAT_LED1
- R2 pad 1: +5V -> /HAT_LED2
- R3 pad 1: +5V -> /HAT_LED3
- R4 pad 1: +5V -> /DEBUG_LED2
- R4 pad 2: unconnected-(R4-Pad2) -> Net-(D4-A)
- U1 pad 1: unconnected-(U1-MCLK-Pad1) -> /I2S_MCK
- U1 pad 17: unconnected-(U1-AVSS1-Pad17) -> GND
- U1 pad 18: unconnected-(U1-DRVDD-Pad18) -> +3.3VA
- U1 pad 2: unconnected-(U1-BCLK-Pad2) -> /I2S_BCK
- U1 pad 21: unconnected-(U1-DRVSS-Pad21) -> GND
- U1 pad 24: unconnected-(U1-DRVDD-Pad24) -> +3.3VA
- U1 pad 25: unconnected-(U1-AVDD-Pad25) -> +3.3VA
- U1 pad 26: unconnected-(U1-AVSS2-Pad26) -> GND
- U1 pad 3: unconnected-(U1-WCLK-Pad3) -> /I2S_WS
- U1 pad 31: unconnected-(U1-*RESET-Pad31) -> /~{CODEC_RESET}
- U1 pad 32: unconnected-(U1-DVDD-Pad32) -> +1.8V
- U1 pad 33: unconnected-(U1-EPAD-Pad33) -> GND
- U1 pad 4: unconnected-(U1-DIN-Pad4) -> /I2S_SD_DAC
- U1 pad 5: unconnected-(U1-DOUT-Pad5) -> /I2S_SD_ADC
- U1 pad 6: unconnected-(U1-DVSS-Pad6) -> GND
- U1 pad 7: unconnected-(U1-IOVDD-Pad7) -> +3.3V
- U1 pad 8: unconnected-(U1-SCL-Pad8) -> /SCL
- U1 pad 9: unconnected-(U1-SDA-Pad9) -> /SDA
- U2 pad 1: unconnected-(U2-PE2-Pad1) -> /STM32F429VIT6/PE2
- U2 pad 10: Net-(U2-VSS-Pad10) -> GND
- U2 pad 100: unconnected-(U2-VDD-Pad100) -> +3.3V
- U2 pad 11: unconnected-(U2-VDD-Pad11) -> +3.3V
- U2 pad 12: unconnected-(U2-PH0-Pad12) -> /STM32F429VIT6/XTAL_IN
- U2 pad 13: unconnected-(U2-PH1-Pad13) -> /STM32F429VIT6/XTAL_OUT
- U2 pad 14: unconnected-(U2-NRST-Pad14) -> /STM32F429VIT6/RESET
- U2 pad 15: unconnected-(U2-PC0-Pad15) -> /STM32F429VIT6/PC0
- U2 pad 16: unconnected-(U2-PC1-Pad16) -> /STM32F429VIT6/PC1
- U2 pad 17: unconnected-(U2-PC2-Pad17) -> /I2S_SD_DAC
- U2 pad 18: unconnected-(U2-PC3-Pad18) -> /I2S_SD_ADC
- U2 pad 19: unconnected-(U2-VDD-Pad19) -> +3.3V
- U2 pad 2: unconnected-(U2-PE3-Pad2) -> /STM32F429VIT6/PE3
- U2 pad 20: unconnected-(U2-VSSA-Pad20) -> GND
- U2 pad 21: unconnected-(U2-VREF+-Pad21) -> Net-(U2-VREF+)
- U2 pad 22: unconnected-(U2-VDDA-Pad22) -> +3.3VA
- U2 pad 23: unconnected-(U2-PA0-Pad23) -> /POT1
- U2 pad 24: unconnected-(U2-PA1-Pad24) -> /POT2
- U2 pad 25: unconnected-(U2-PA2-Pad25) -> /POT3
- U2 pad 26: unconnected-(U2-PA3-Pad26) -> /POT4
- U2 pad 27: Net-(U2-VSS-Pad10) -> GND
- U2 pad 28: unconnected-(U2-VDD-Pad28) -> +3.3V
- U2 pad 29: unconnected-(U2-PA4-Pad29) -> /STM32F429VIT6/DAC_OUT1
- U2 pad 3: unconnected-(U2-PE4-Pad3) -> /STM32F429VIT6/PE4
- U2 pad 30: unconnected-(U2-PA5-Pad30) -> /STM32F429VIT6/DAC_OUT2
- U2 pad 31: unconnected-(U2-PA6-Pad31) -> /LED_DIN
- U2 pad 32: unconnected-(U2-PA7-Pad32) -> /DEBUG_LED1
- U2 pad 33: unconnected-(U2-PC4-Pad33) -> /STM32F429VIT6/PC4
- U2 pad 34: unconnected-(U2-PC5-Pad34) -> /STM32F429VIT6/PC5
- U2 pad 35: unconnected-(U2-PB0-Pad35) -> /HAT_LED1
- U2 pad 36: unconnected-(U2-PB1-Pad36) -> /HAT_LED2
- U2 pad 37: unconnected-(U2-PB2-Pad37) -> /HAT_LED3
- U2 pad 38: unconnected-(U2-PE7-Pad38) -> /STM32F429VIT6/PE7
- U2 pad 39: unconnected-(U2-PE8-Pad39) -> /STM32F429VIT6/PE8
- U2 pad 4: unconnected-(U2-PE5-Pad4) -> /STM32F429VIT6/PE5
- U2 pad 40: unconnected-(U2-PE9-Pad40) -> /STM32F429VIT6/PE9
- U2 pad 41: unconnected-(U2-PE10-Pad41) -> /STM32F429VIT6/PE10
- U2 pad 42: unconnected-(U2-PE11-Pad42) -> /STM32F429VIT6/PE11
- U2 pad 43: unconnected-(U2-PE12-Pad43) -> /STM32F429VIT6/PE12
- U2 pad 44: unconnected-(U2-PE13-Pad44) -> /STM32F429VIT6/PE13
- U2 pad 45: unconnected-(U2-PE14-Pad45) -> /STM32F429VIT6/PE14
- U2 pad 46: unconnected-(U2-PE15-Pad46) -> /STM32F429VIT6/PE15
- U2 pad 47: unconnected-(U2-PB10-Pad47) -> /I2S_BCK
- U2 pad 48: unconnected-(U2-PB11-Pad48) -> /STM32F429VIT6/PB11
- U2 pad 49: unconnected-(U2-VCAP_1-Pad49) -> Net-(U2-VCAP_1)
- U2 pad 5: unconnected-(U2-PE6-Pad5) -> /STM32F429VIT6/PE6
- U2 pad 50: unconnected-(U2-VDD-Pad50) -> +3.3V
- U2 pad 51: unconnected-(U2-PB12-Pad51) -> /I2S_WS
- U2 pad 52: unconnected-(U2-PB13-Pad52) -> /STM32F429VIT6/PB13
- U2 pad 53: unconnected-(U2-PB14-Pad53) -> /STM32F429VIT6/PB14
- U2 pad 54: unconnected-(U2-PB15-Pad54) -> /STM32F429VIT6/PB15
- U2 pad 55: unconnected-(U2-PD8-Pad55) -> /STM32F429VIT6/PD8
- U2 pad 56: unconnected-(U2-PD9-Pad56) -> /STM32F429VIT6/PD9
- U2 pad 57: unconnected-(U2-PD10-Pad57) -> /STM32F429VIT6/PD10
- U2 pad 58: unconnected-(U2-PD11-Pad58) -> /STM32F429VIT6/PD11
- U2 pad 59: unconnected-(U2-PD12-Pad59) -> /STM32F429VIT6/PD12
- U2 pad 60: unconnected-(U2-PD13-Pad60) -> /STM32F429VIT6/PD13
- U2 pad 61: unconnected-(U2-PD14-Pad61) -> /STM32F429VIT6/PD14
- U2 pad 62: unconnected-(U2-PD15-Pad62) -> /STM32F429VIT6/PD15
- U2 pad 63: unconnected-(U2-PC6-Pad63) -> /I2S_MCK
- U2 pad 64: unconnected-(U2-PC7-Pad64) -> /STM32F429VIT6/PC7
- U2 pad 65: unconnected-(U2-PC8-Pad65) -> /STM32F429VIT6/PC8
- U2 pad 66: unconnected-(U2-PC9-Pad66) -> /STM32F429VIT6/PC9
- U2 pad 67: unconnected-(U2-PA8-Pad67) -> /DEBUG_LED2
- U2 pad 68: unconnected-(U2-PA9-Pad68) -> /UART_TX
- U2 pad 69: unconnected-(U2-PA10-Pad69) -> /UART_RX
- U2 pad 7: unconnected-(U2-PC13-Pad7) -> /STM32F429VIT6/PC13
- U2 pad 70: unconnected-(U2-PA11-Pad70) -> /USB_D-
- U2 pad 71: unconnected-(U2-PA12-Pad71) -> /USB_D+
- U2 pad 72: unconnected-(U2-PA13-Pad72) -> /STM32F429VIT6/SWDIO
- U2 pad 73: unconnected-(U2-VCAP_2-Pad73) -> Net-(U2-VCAP_2)
- U2 pad 74: Net-(U2-VSS-Pad10) -> GND
- U2 pad 75: unconnected-(U2-VDD-Pad75) -> +3.3V
- U2 pad 76: unconnected-(U2-PA14-Pad76) -> /STM32F429VIT6/SWCLCK
- U2 pad 77: unconnected-(U2-PA15-Pad77) -> /DEBUG_LED3
- U2 pad 78: unconnected-(U2-PC10-Pad78) -> /STM32F429VIT6/PC10
- U2 pad 79: unconnected-(U2-PC11-Pad79) -> /STM32F429VIT6/PC11
- U2 pad 8: unconnected-(U2-PC14-Pad8) -> /STM32F429VIT6/PC14
- U2 pad 80: unconnected-(U2-PC12-Pad80) -> /STM32F429VIT6/PC12
- U2 pad 81: unconnected-(U2-PD0-Pad81) -> /STM32F429VIT6/PD0
- U2 pad 82: unconnected-(U2-PD1-Pad82) -> /STM32F429VIT6/PD1
- U2 pad 83: unconnected-(U2-PD2-Pad83) -> /STM32F429VIT6/PD2
- U2 pad 84: unconnected-(U2-PD3-Pad84) -> /STM32F429VIT6/PD3
- U2 pad 85: unconnected-(U2-PD4-Pad85) -> /STM32F429VIT6/PD4
- U2 pad 86: unconnected-(U2-PD5-Pad86) -> /STM32F429VIT6/PD5
- U2 pad 87: unconnected-(U2-PD6-Pad87) -> /STM32F429VIT6/PD6
- U2 pad 88: unconnected-(U2-PD7-Pad88) -> /STM32F429VIT6/PD7
- U2 pad 89: unconnected-(U2-PB3-Pad89) -> /~{CODEC_RESET}
- U2 pad 9: unconnected-(U2-PC15-Pad9) -> /STM32F429VIT6/PC15
- U2 pad 90: unconnected-(U2-PB4-Pad90) -> /STM32F429VIT6/PB4
- U2 pad 91: unconnected-(U2-PB5-Pad91) -> /STM32F429VIT6/PB5
- U2 pad 92: unconnected-(U2-PB6-Pad92) -> /SDA
- U2 pad 93: unconnected-(U2-PB7-Pad93) -> /SCL
- U2 pad 94: unconnected-(U2-BOOT0-Pad94) -> Net-(U2-BOOT0)
- U2 pad 95: unconnected-(U2-PB8-Pad95) -> /STM32F429VIT6/PB8
- U2 pad 96: unconnected-(U2-PB9-Pad96) -> /STM32F429VIT6/PB9
- U2 pad 97: unconnected-(U2-PE0-Pad97) -> /STM32F429VIT6/PE0
- U2 pad 98: unconnected-(U2-PE1-Pad98) -> /STM32F429VIT6/PE1
- U2 pad 99: Net-(U2-VSS-Pad10) -> GND
Other:
- board size 49.1 x 106.6 mm -> 63.8 x 138.6 mm
- copper layers 2 -> 4

Commit message: more schematic stuff, preliminary footprint choices and parts grouping, played with multicahnnel for the buttons
Parts:
- removed the C16 at (142.5, 83.5)
- removed the C17 at (137.5, 87.0)
- removed the C18 at (142.5, 89.3)
- removed the C2 at (133.5, 82.0)
- removed the J1 at (155.5, 157.8)
- removed the J2 at (126.5, 155.0)
- removed the U3 at (130.0, 62.0)
- added C10: 2.2u, Capacitor_SMD:C_0603_1608Metric, F.Cu at (82.2, 121.9)
- added C11: 47u, Capacitor_SMD:CP_Elec_4x3, F.Cu at (88.1, 124.4)
- added C3: 10n, Capacitor_SMD:C_0603_1608Metric, F.Cu at (199.0, 87.0)
- added C35: 220p, Capacitor_SMD:C_0603_1608Metric, F.Cu at (22.4, 143.9)
- added C36: 10n, Capacitor_SMD:C_0603_1608Metric, F.Cu at (22.4, 146.4)
- added C37: 10u, Capacitor_SMD:C_0603_1608Metric, F.Cu at (22.4, 148.9)
- added C38: 100n, Capacitor_SMD:C_0603_1608Metric, F.Cu at (22.4, 151.4)
- added C39: 100n, Capacitor_SMD:C_0603_1608Metric, F.Cu at (22.4, 153.9)
- added C4: 1u, Capacitor_SMD:CP_Elec_4x3, F.Cu at (193.1, 88.7)
- added C40: 100n, Capacitor_SMD:C_0603_1608Metric, F.Cu at (22.4, 156.4)
- added C41: 10u, Capacitor_SMD:C_0603_1608Metric, F.Cu at (22.4, 158.9)
- added C42: 10u, Capacitor_SMD:C_0603_1608Metric, F.Cu at (22.4, 161.4)
- added C43: 10u, Capacitor_SMD:C_0603_1608Metric, F.Cu at (22.4, 164.0)
- added C44: 2.2u, Diode_SMD:D_SOD-123, B.Cu at (-4.41, 76.4)
- added C45: 2.2u, Diode_SMD:D_SOD-123, B.Cu at (13.6, 72.7)
- added C46: 2.2u, Diode_SMD:D_SOD-123, B.Cu at (49.7, 78.1)
- added C47: 2.2u, Diode_SMD:D_SOD-123, B.Cu at (7.62, 94.3)
- added C48: 2.2u, Diode_SMD:D_SOD-123, B.Cu at (37.7, 78.9)
- added C49: 2.2u, Diode_SMD:D_SOD-123, B.Cu at (19.6, 59.4)
- added C5: 100n, Capacitor_SMD:C_0603_1608Metric, F.Cu at (199.0, 89.5)
- added C50: 220p, Capacitor_SMD:C_0603_1608Metric, F.Cu at (53.3, 144.5)
- added C51: 10n, Capacitor_SMD:C_0603_1608Metric, F.Cu at (53.3, 147.0)
- added C52: 10u, Capacitor_SMD:C_0603_1608Metric, F.Cu at (53.3, 149.5)
- added C53: 100n, Capacitor_SMD:C_0603_1608Metric, F.Cu at (53.3, 152.0)
- added C54: 100n, Capacitor_SMD:C_0603_1608Metric, F.Cu at (53.3, 154.5)
- added C55: 100n, Capacitor_SMD:C_0603_1608Metric, F.Cu at (53.3, 157.0)
- added C56: 10u, Capacitor_SMD:C_0603_1608Metric, F.Cu at (53.3, 159.6)
- added C57: 10u, Capacitor_SMD:C_0603_1608Metric, F.Cu at (53.3, 162.1)
- added C58: 10u, Capacitor_SMD:C_0603_1608Metric, F.Cu at (53.3, 164.6)
- added C59: 2.2u, Diode_SMD:D_SOD-123, B.Cu at (31.7, 60.9)
- added C6: 1u, Capacitor_SMD:CP_Elec_4x3, F.Cu at (193.1, 94.5)
- added C60: 2.2u, Diode_SMD:D_SOD-123, B.Cu at (43.7, 61.4)
- added C61: 2.2u, Diode_SMD:D_SOD-123, B.Cu at (1.60, 59.9)
- added C62: 2.2u, Diode_SMD:D_SOD-123, B.Cu at (-16.4, 77.5)
- added C63: 2.2u, Diode_SMD:D_SOD-123, B.Cu at (-10.4, 63.5)
- added C64: 2.2u, Diode_SMD:D_SOD-123, B.Cu at (25.7, 94.3)
- added C7: 2.2u, Capacitor_SMD:C_0603_1608Metric, F.Cu at (82.2, 114.4)
- added C8: 2.2u, Capacitor_SMD:C_0603_1608Metric, F.Cu at (82.2, 116.9)
- added C9: 1u, Capacitor_SMD:C_0603_1608Metric, F.Cu at (82.2, 119.4)
- added D10: D_Schottky, Diode_SMD:D_SOD-123, F.Cu at (94.9, 126.5)
- added D11: CG0402MLU-12G, Diode_SMD:D_SOD-123, F.Cu at (31.7, 158.5)
- added D12: D_Schottky, Diode_SMD:D_SOD-123, F.Cu at (31.7, 161.8)
- added D13: 1N4148, Diode_SMD:D_SOD-123, B.Cu at (-1.91, 76.4)
- added D14: 1N4148, Diode_SMD:D_SOD-123, B.Cu at (16.1, 72.7)
- added D15: 1N4148, Diode_SMD:D_SOD-123, B.Cu at (52.2, 78.1)
- added D16: 1N4148, Diode_SMD:D_SOD-123, B.Cu at (10.1, 94.3)
- added D17: 1N4148, Diode_SMD:D_SOD-123, B.Cu at (40.2, 78.9)
- added D18: 1N4148, Diode_SMD:D_SOD-123, B.Cu at (22.1, 59.4)
- added D19: CG0402MLU-12G, Diode_SMD:D_SOD-123, F.Cu at (62.6, 159.1)
- added D20: D_Schottky, Diode_SMD:D_SOD-123, F.Cu at (62.6, 162.5)
- added D21: 1N4148, Diode_SMD:D_SOD-123, B.Cu at (34.2, 60.9)
- added D22: 1N4148, Diode_SMD:D_SOD-123, B.Cu at (46.2, 61.4)
- added D23: 1N4148, Diode_SMD:D_SOD-123, B.Cu at (4.10, 59.9)
- added D24: 1N4148, Diode_SMD:D_SOD-123, B.Cu at (-13.9, 77.5)
- added D25: 1N4148, Diode_SMD:D_SOD-123, B.Cu at (-7.92, 63.5)
- added D26: 1N4148, Diode_SMD:D_SOD-123, B.Cu at (28.2, 94.3)
- added D6: WS2812, LED_SMD:LED_WS2812_PLCC6_5.0x5.0mm_P1.6mm, F.Cu at (-42.0, 72.7)
- added D9: D_Schottky, Diode_SMD:D_SOD-123, F.Cu at (94.9, 123.1)
- added FB2: 120R, Resistor_SMD:R_0603_1608Metric, F.Cu at (82.2, 124.4)
- added J3: Conn_01x03_Socket, Connector_JST:JST_ZE_B03B-ZESK-1D_1x03_P1.50mm_Vertical, F.Cu at (123.5, 188.2)
- added J4: Conn_01x03_Socket, Connector_JST:JST_ZE_B03B-ZESK-1D_1x03_P1.50mm_Vertical, F.Cu at (134.5, 188.0)
- added R14: 100R, Resistor_SMD:R_0603_1608Metric_Pad0.98x0.95mm_HandSolder, F.Cu at (26.6, 143.9)
- added R15: 1M, Resistor_SMD:R_0603_1608Metric_Pad0.98x0.95mm_HandSolder, F.Cu at (26.6, 146.4)
- added R16: 1M, Resistor_SMD:R_0603_1608Metric_Pad0.98x0.95mm_HandSolder, F.Cu at (26.6, 148.9)
- added R17: 1k, Resistor_SMD:R_0603_1608Metric_Pad0.98x0.95mm_HandSolder, F.Cu at (26.6, 151.4)
- added R18: 1M, Resistor_SMD:R_0603_1608Metric_Pad0.98x0.95mm_HandSolder, F.Cu at (26.6, 153.9)
- added R19: 100, Resistor_SMD:R_0603_1608Metric_Pad0.98x0.95mm_HandSolder, F.Cu at (26.6, 156.4)
- added R20: 1k, Resistor_SMD:R_0603_1608Metric_Pad0.98x0.95mm_HandSolder, F.Cu at (26.6, 158.9)
- added R21: 1k, Resistor_SMD:R_0603_1608Metric_Pad0.98x0.95mm_HandSolder, F.Cu at (26.6, 161.4)
- added R22: 2.26k 1%, Resistor_SMD:R_0603_1608Metric_Pad0.98x0.95mm_HandSolder, B.Cu at (-3.21, 79.9)
- added R23: 2.05k 1%, Resistor_SMD:R_0603_1608Metric_Pad0.98x0.95mm_HandSolder, B.Cu at (0.09, 76.9)
- added R24: 2.26k 1%, Resistor_SMD:R_0603_1608Metric_Pad0.98x0.95mm_HandSolder, B.Cu at (14.8, 76.2)
- added R25: 2.05k 1%, Resistor_SMD:R_0603_1608Metric_Pad0.98x0.95mm_HandSolder, B.Cu at (18.1, 73.2)
- added R26: 2.26k 1%, Resistor_SMD:R_0603_1608Metric_Pad0.98x0.95mm_HandSolder, B.Cu at (50.9, 81.6)
- added R27: 2.05k 1%, Resistor_SMD:R_0603_1608Metric_Pad0.98x0.95mm_HandSolder, B.Cu at (54.2, 78.6)
- added R28: 2.26k 1%, Resistor_SMD:R_0603_1608Metric_Pad0.98x0.95mm_HandSolder, B.Cu at (8.81, 97.8)
- added R29: 2.05k 1%, Resistor_SMD:R_0603_1608Metric_Pad0.98x0.95mm_HandSolder, B.Cu at (12.1, 94.8)
- added R30: 2.26k 1%, Resistor_SMD:R_0603_1608Metric_Pad0.98x0.95mm_HandSolder, B.Cu at (38.9, 82.4)
- added R31: 2.05k 1%, Resistor_SMD:R_0603_1608Metric_Pad0.98x0.95mm_HandSolder, B.Cu at (42.2, 79.4)
- added R32: 2.26k 1%, Resistor_SMD:R_0603_1608Metric_Pad0.98x0.95mm_HandSolder, B.Cu at (20.8, 62.9)
- added R33: 2.05k 1%, Resistor_SMD:R_0603_1608Metric_Pad0.98x0.95mm_HandSolder, B.Cu at (24.1, 59.9)
- added R34: 100R, Resistor_SMD:R_0603_1608Metric_Pad0.98x0.95mm_HandSolder, F.Cu at (57.5, 144.5)
- added R35: 1M, Resistor_SMD:R_0603_1608Metric_Pad0.98x0.95mm_HandSolder, F.Cu at (57.5, 147.0)
- added R36: 1M, Resistor_SMD:R_0603_1608Metric_Pad0.98x0.95mm_HandSolder, F.Cu at (57.5, 149.5)
- added R37: 1k, Resistor_SMD:R_0603_1608Metric_Pad0.98x0.95mm_HandSolder, F.Cu at (57.5, 152.0)
- added R38: 1M, Resistor_SMD:R_0603_1608Metric_Pad0.98x0.95mm_HandSolder, F.Cu at (57.5, 154.5)
- added R39: 100, Resistor_SMD:R_0603_1608Metric_Pad0.98x0.95mm_HandSolder, F.Cu at (57.5, 157.0)
- added R40: 1k, Resistor_SMD:R_0603_1608Metric_Pad0.98x0.95mm_HandSolder, F.Cu at (57.5, 159.6)
- added R41: 1k, Resistor_SMD:R_0603_1608Metric_Pad0.98x0.95mm_HandSolder, F.Cu at (57.5, 162.1)
- added R42: 2.26k 1%, Resistor_SMD:R_0603_1608Metric_Pad0.98x0.95mm_HandSolder, B.Cu at (32.9, 64.4)
- added R43: 2.05k 1%, Resistor_SMD:R_0603_1608Metric_Pad0.98x0.95mm_HandSolder, B.Cu at (36.2, 61.4)
- added R44: 2.26k 1%, Resistor_SMD:R_0603_1608Metric_Pad0.98x0.95mm_HandSolder, B.Cu at (44.9, 64.9)
- added R45: 2.05k 1%, Resistor_SMD:R_0603_1608Metric_Pad0.98x0.95mm_HandSolder, B.Cu at (48.2, 61.9)
- added R46: 2.26k 1%, Resistor_SMD:R_0603_1608Metric_Pad0.98x0.95mm_HandSolder, B.Cu at (2.80, 63.4)
- added R47: 2.05k 1%, Resistor_SMD:R_0603_1608Metric_Pad0.98x0.95mm_HandSolder, B.Cu at (6.10, 60.4)
- added R48: 2.26k 1%, Resistor_SMD:R_0603_1608Metric_Pad0.98x0.95mm_HandSolder, B.Cu at (-15.2, 81.0)
- added R49: 2.05k 1%, Resistor_SMD:R_0603_1608Metric_Pad0.98x0.95mm_HandSolder, B.Cu at (-11.9, 78.0)
- added R50: 2.26k 1%, Resistor_SMD:R_0603_1608Metric_Pad0.98x0.95mm_HandSolder, B.Cu at (-9.22, 67.0)
- added R51: 2.05k 1%, Resistor_SMD:R_0603_1608Metric_Pad0.98x0.95mm_HandSolder, B.Cu at (-5.92, 64.0)
- added R52: 2.26k 1%, Resistor_SMD:R_0603_1608Metric_Pad0.98x0.95mm_HandSolder, B.Cu at (26.8, 97.8)
- added R53: 2.05k 1%, Resistor_SMD:R_0603_1608Metric_Pad0.98x0.95mm_HandSolder, B.Cu at (30.2, 94.8)
- added R7: 1k, Resistor_SMD:R_0603_1608Metric_Pad0.98x0.95mm_HandSolder, F.Cu at (96.3, 114.4)
- added R8: 1k, Resistor_SMD:R_0603_1608Metric_Pad0.98x0.95mm_HandSolder, F.Cu at (96.3, 116.9)
- added RV5: 12V, Varistor:RV_Disc_D7mm_W3.4mm_P5mm, F.Cu at (30.6, 153.7)
- added RV6: 12V, Varistor:RV_Disc_D7mm_W3.4mm_P5mm, F.Cu at (61.5, 154.3)
- added SW10: SW_Push, Button_Switch_SMD:SW_SPST_PTS645, F.Cu at (44.9, 61.7)
- added SW11: SW_Push, Button_Switch_SMD:SW_SPST_PTS645, F.Cu at (2.80, 60.2)
- added SW12: SW_Push, Button_Switch_SMD:SW_SPST_PTS645, F.Cu at (-15.2, 77.8)
- added SW13: SW_Push, Button_Switch_SMD:SW_SPST_PTS645, F.Cu at (-9.22, 63.8)
- added SW14: SW_Push, Button_Switch_SMD:SW_SPST_PTS645, F.Cu at (26.8, 94.7)
- added SW3: SW_Push, Button_Switch_SMD:SW_SPST_PTS645, F.Cu at (-3.21, 76.7)
- added SW4: SW_Push, Button_Switch_SMD:SW_SPST_PTS645, F.Cu at (14.8, 73.0)
- added SW5: SW_Push, Button_Switch_SMD:SW_SPST_PTS645, F.Cu at (50.9, 78.4)
- added SW6: SW_Push, Button_Switch_SMD:SW_SPST_PTS645, F.Cu at (8.81, 94.6)
- added SW7: SW_Push, Button_Switch_SMD:SW_SPST_PTS645, F.Cu at (38.9, 79.2)
- added SW8: SW_Push, Button_Switch_SMD:SW_SPST_PTS645, F.Cu at (20.8, 59.7)
- added SW9: SW_Push, Button_Switch_SMD:SW_SPST_PTS645, F.Cu at (32.9, 61.2)
- added U1: TLV76133DCY, Package_TO_SOT_SMD:SOT-223-3_TabPin2, F.Cu at (131.5, 62.5)
- added U10: 74HC14, Package_SO:SO-14_3.9x8.65mm_P1.27mm, F.Cu at (17.5, 46.2)
- added U2: TLV76150DCY, Package_TO_SOT_SMD:SOT-223-3_TabPin2, F.Cu at (89.2, 117.3)
- added U5: TLV9061xDBV, Package_TO_SOT_SMD:SOT-23-5, F.Cu at (31.4, 145.0)
- added U6: TLV9061xDBV, Package_TO_SOT_SMD:SOT-23-5, F.Cu at (31.4, 149.6)
- added U7: 74HC14, Package_SO:SO-14_3.9x8.65mm_P1.27mm, F.Cu at (-7.58, 93.2)
- added U8: TLV9061xDBV, Package_TO_SOT_SMD:SOT-23-5, F.Cu at (62.3, 145.6)
- added U9: TLV9061xDBV, Package_TO_SOT_SMD:SOT-23-5, F.Cu at (62.3, 150.3)
- C1: renamed from C4; value 10u -> 1u
- C2: renamed from C7; value 10u -> 2.2u
- FB1: moved to F.Cu
- SW2: renamed from SW1; footprint Button_Switch_SMD:Panasonic_EVQPUK_EVQPUB -> Button_Switch_SMD:SW_SPST_PTS645
- moved FB1 61.5 mm to (199.0, 92.0), turned to 0 degrees
- renumbered C23 to C12, C19 to C13, C24 to C14, C20 to C15, C25 to C16, C21 to C17, C26 to C18, C22 to C19, C27 to C20, C28 to C21, C29 to C22, C1 to C23, C3 to C24, C9 to C25, C5 to C26, C6 to C27, C13 to C28, C8 to C29, C10 to C30, C11 to C31, C14 to C32, C15 to C33, C12 to C34, D6 to D1, D1 to D2, D5 to D3, D2 to D5, D3 to D8, J4 to J1, J5 to J2, J3 to J5, R10 to R1, R9 to R10, R7 to R11, R5 to R12, R6 to R13, R1 to R2, R4 to R3, R2 to R4, R11 to R5, R3 to R6, R8 to R9, SW2 to SW1, U1 to U3, U2 to U4
Connections:
- net /STM32F429VIT6/PE0 renamed /C
- net /STM32F429VIT6/PE1 renamed /C#
- net /STM32F429VIT6/PE10 renamed /A#
- net /STM32F429VIT6/PE11 renamed /B
- net /STM32F429VIT6/PE2 renamed /D
- net /STM32F429VIT6/PE3 renamed /D#
- net /STM32F429VIT6/PE4 renamed /E
- net /STM32F429VIT6/PE5 renamed /F
- net /STM32F429VIT6/PE6 renamed /F#
- net /STM32F429VIT6/PE7 renamed /G
- net /STM32F429VIT6/PE8 renamed /G#
- net /STM32F429VIT6/PE9 renamed /A
- D3 pad 1: /LED_DOUT -> Net-(D3-DOUT)
- U3 pad 10: unconnected-(U1-MIC1L/LINE1L-Pad10) -> /BUFFERED_AUDIO_INPUT_L
- U3 pad 11: unconnected-(U1-MIC1R/LINE1R-Pad11) -> /BUFFERED_AUDIO_INPUT_R
- U3 pad 27: unconnected-(U1-LEFT_LOP-Pad27) -> /CODEC_AUDIO_OUTPUT_L
- U3 pad 28: unconnected-(U1-LEFT_LOM-Pad28) -> /CODEC_AUDIO_OUTPUT_L_MINUS
- U3 pad 29: unconnected-(U1-RIGHT_LOP-Pad29) -> /CODEC_AUDIO_OUTPUT_R
- U3 pad 30: unconnected-(U1-RIGHT_LOM-Pad30) -> /CODEC_AUDIO_OUTPUT_R_MINUS
- U4 pad 81: /STM32F429VIT6/PD0 -> /OCTAVE_UP
- U4 pad 82: /STM32F429VIT6/PD1 -> /OCTAVE_DOWN
- U4 pad 83: /STM32F429VIT6/PD2 -> /LEFT
- U4 pad 84: /STM32F429VIT6/PD3 -> /RIGHT
- U4 pad 85: /STM32F429VIT6/PD4 -> /UP
- U4 pad 86: /STM32F429VIT6/PD5 -> /DOWN
Routing:
- net GND: track 0.00 -> 158.4 mm, vias 0 -> 12
- net Net-(D24-A): track 0.00 -> 14.4 mm, vias 0 -> 1
- net Net-(D26-A): track 0.00 -> 14.4 mm, vias 0 -> 1
- net Net-(D25-A): track 0.00 -> 14.4 mm, vias 0 -> 1
- net Net-(D21-A): track 0.00 -> 14.4 mm, vias 0 -> 1
- net Net-(D23-A): track 0.00 -> 14.4 mm, vias 0 -> 1
- net Net-(D18-A): track 0.00 -> 14.4 mm, vias 0 -> 1
- net Net-(D22-A): track 0.00 -> 14.4 mm, vias 0 -> 1
- net Net-(D15-A): track 0.00 -> 14.4 mm, vias 0 -> 1
- net Net-(D17-A): track 0.00 -> 14.4 mm, vias 0 -> 1
- net Net-(D16-A): track 0.00 -> 14.4 mm, vias 0 -> 1
- net Net-(D14-A): track 0.00 -> 14.4 mm, vias 0 -> 1
- net Net-(D13-A): track 0.00 -> 14.4 mm, vias 0 -> 1
- net /Keys/Debounced Button2/OUT_TO_SCHMIDT_TRIGGER: track 0.00 -> 5.42 mm
- net /Buttons/Debounced Button3/OUT_TO_SCHMIDT_TRIGGER: track 0.00 -> 5.42 mm
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
Commit message: expand usb, piano keys, cleanup
Parts:
- removed the C1 at (131.5, 56.0)
- removed the C2 at (128.2, 68.0)
- removed the C3 at (199.0, 87.0)
- removed the C4 at (193.1, 88.7)
- removed the C44 at (-4.41, 76.4)
- removed the C45 at (13.6, 72.7)
- removed the C46 at (49.7, 78.1)
- removed the C47 at (7.62, 94.3)
- removed the C48 at (37.7, 78.9)
- removed the C49 at (19.6, 59.4)
- removed the C5 at (199.0, 89.5)
- removed the C6 at (193.1, 94.5)
- removed the D13 at (-1.91, 76.4)
- removed the D14 at (16.1, 72.7)
- removed the FB1 at (199.0, 92.0)
- removed P1: USB_C_Plug_USB2.0, Connector_USB:USB_C_Receptacle_GCT_USB4105-xx-A_16P_TopMnt_Horizontal
- removed the R22 at (-3.21, 79.9)
- removed the R23 at (0.09, 76.9)
- removed the R24 at (14.8, 76.2)
- removed the R25 at (18.1, 73.2)
- removed the R26 at (50.9, 81.6)
- removed the R27 at (54.2, 78.6)
- removed the R28 at (8.81, 97.8)
- removed the R29 at (12.1, 94.8)
- removed the U1 at (131.5, 62.5)
- removed the U7 at (-7.58, 93.2)
- added C19: 10n, Capacitor_SMD:C_0603_1608Metric, F.Cu at (-50.3, 124.5)
- added C22: 1u, Capacitor_SMD:CP_Elec_4x3, F.Cu at (-56.2, 126.2)
- added C26: 100n, Capacitor_SMD:C_0603_1608Metric, F.Cu at (-50.3, 127.0)
- added C28: 1u, Capacitor_SMD:CP_Elec_4x3, F.Cu at (-56.2, 132.0)
- added C51: 100uF, Capacitor_SMD:C_1206_3216Metric, F.Cu at (-108.8, 62.8)
- added C52: 100uF, Capacitor_SMD:C_1206_3216Metric, F.Cu at (-108.8, 66.2)
- added C53: 100uF, Capacitor_SMD:C_1206_3216Metric, F.Cu at (-108.8, 69.5)
- added C54: 100uF, Capacitor_SMD:C_1206_3216Metric, F.Cu at (-108.8, 72.9)
- added C55: 1u, Capacitor_SMD:CP_Elec_4x3, F.Cu at (-115.5, 64.1)
- added C56: 2.2u, Capacitor_SMD:CP_Elec_4x3, F.Cu at (-115.5, 69.9)
- added C57: 2.2u, Diode_SMD:D_SOD-123, F.Cu at (-94.0, -25.8)
- added C58: 2.2u, Diode_SMD:D_SOD-123, F.Cu at (-94.0, -22.4)
- added C65: 2.2u, Diode_SMD:D_SOD-123, F.Cu at (17.1, 53.6)
- added C66: 2.2u, Diode_SMD:D_SOD-123, F.Cu at (17.1, 56.9)
- added C67: 2.2u, Diode_SMD:D_SOD-123, F.Cu at (17.1, 60.3)
- added C68: 2.2u, Diode_SMD:D_SOD-123, F.Cu at (17.1, 63.6)
- added C69: 2.2u, Diode_SMD:D_SOD-123, F.Cu at (22.9, 46.9)
- added C70: 2.2u, Diode_SMD:D_SOD-123, F.Cu at (22.9, 50.2)
- added C71: 2.2u, Diode_SMD:D_SOD-123, F.Cu at (22.9, 53.6)
- added C72: 2.2u, Diode_SMD:D_SOD-123, F.Cu at (22.9, 56.9)
- added C73: 2.2u, Diode_SMD:D_SOD-123, F.Cu at (22.9, 60.3)
- added C74: 2.2u, Diode_SMD:D_SOD-123, F.Cu at (22.9, 63.6)
- added D19: 1N4148, Diode_SMD:D_SOD-123, F.Cu at (-82.4, -19.1)
- added D20: 1N4148, Diode_SMD:D_SOD-123, F.Cu at (-82.4, -15.7)
- added D27: 1N4148, Diode_SMD:D_SOD-123, F.Cu at (34.5, 46.9)
- added D28: 1N4148, Diode_SMD:D_SOD-123, F.Cu at (34.5, 50.2)
- added D29: 1N4148, Diode_SMD:D_SOD-123, F.Cu at (34.5, 53.6)
- added D30: 1N4148, Diode_SMD:D_SOD-123, F.Cu at (34.5, 56.9)
- added D31: 1N4148, Diode_SMD:D_SOD-123, F.Cu at (34.5, 60.3)
- added D32: 1N4148, Diode_SMD:D_SOD-123, F.Cu at (34.5, 63.6)
- added F1: SL1206150, Fuse:Fuse_1206_3216Metric_Pad1.42x1.75mm_HandSolder, F.Cu at (-103.0, 67.4)
- added FB2: 120R, Resistor_SMD:R_0603_1608Metric, F.Cu at (-50.3, 129.5)
- added J1: Conn_01x03_Socket, Connector_JST:JST_ZE_B03B-ZESK-1D_1x03_P1.50mm_Vertical, F.Cu at (-106.6, 134.5)
- added J7: USB_C_Receptacle_USB2.0_16P, Connector_USB:USB_C_Receptacle_HRO_TYPE-C-31-M-12, F.Cu at (-113.5, 56.5)
- added R34: 2.26k 1%, Resistor_SMD:R_0603_1608Metric_Pad0.98x0.95mm_HandSolder, F.Cu at (-94.8, -7.75)
- added R35: 2.05k 1%, Resistor_SMD:R_0603_1608Metric_Pad0.98x0.95mm_HandSolder, F.Cu at (-94.8, -5.24)
- added R36: 2.26k 1%, Resistor_SMD:R_0603_1608Metric_Pad0.98x0.95mm_HandSolder, F.Cu at (-90.4, -12.8)
- added R37: 2.05k 1%, Resistor_SMD:R_0603_1608Metric_Pad0.98x0.95mm_HandSolder, F.Cu at (-90.4, -10.3)
- added R38: 2.26k 1%, Resistor_SMD:R_0603_1608Metric_Pad0.98x0.95mm_HandSolder, F.Cu at (-90.4, -7.75)
- added R39: 2.05k 1%, Resistor_SMD:R_0603_1608Metric_Pad0.98x0.95mm_HandSolder, F.Cu at (-90.4, -5.24)
- added R40: 2.26k 1%, Resistor_SMD:R_0603_1608Metric_Pad0.98x0.95mm_HandSolder, F.Cu at (-86.1, -12.8)
- added R41: 2.05k 1%, Resistor_SMD:R_0603_1608Metric_Pad0.98x0.95mm_HandSolder, F.Cu at (-86.1, -10.3)
- added R54: 2.26k 1%, Resistor_SMD:R_0603_1608Metric_Pad0.98x0.95mm_HandSolder, F.Cu at (43.9, 56.5)
- added R55: 2.05k 1%, Resistor_SMD:R_0603_1608Metric_Pad0.98x0.95mm_HandSolder, F.Cu at (43.9, 59.0)
- added R56: 2.26k 1%, Resistor_SMD:R_0603_1608Metric_Pad0.98x0.95mm_HandSolder, F.Cu at (48.2, 46.5)
- added R57: 2.05k 1%, Resistor_SMD:R_0603_1608Metric_Pad0.98x0.95mm_HandSolder, F.Cu at (48.2, 49.0)
- added R58: 2.26k 1%, Resistor_SMD:R_0603_1608Metric_Pad0.98x0.95mm_HandSolder, F.Cu at (48.2, 51.5)
- added R59: 2.05k 1%, Resistor_SMD:R_0603_1608Metric_Pad0.98x0.95mm_HandSolder, F.Cu at (48.2, 54.0)
- added R60: 2.26k 1%, Resistor_SMD:R_0603_1608Metric_Pad0.98x0.95mm_HandSolder, F.Cu at (48.2, 56.5)
- added R61: 2.05k 1%, Resistor_SMD:R_0603_1608Metric_Pad0.98x0.95mm_HandSolder, F.Cu at (48.2, 59.0)
- added R62: 2.26k 1%, Resistor_SMD:R_0603_1608Metric_Pad0.98x0.95mm_HandSolder, F.Cu at (52.6, 46.5)
- added R63: 2.05k 1%, Resistor_SMD:R_0603_1608Metric_Pad0.98x0.95mm_HandSolder, F.Cu at (52.6, 49.0)
- added R64: 2.26k 1%, Resistor_SMD:R_0603_1608Metric_Pad0.98x0.95mm_HandSolder, F.Cu at (52.6, 51.5)
- added R65: 2.05k 1%, Resistor_SMD:R_0603_1608Metric_Pad0.98x0.95mm_HandSolder, F.Cu at (52.6, 54.0)
- added R66: 2.26k 1%, Resistor_SMD:R_0603_1608Metric_Pad0.98x0.95mm_HandSolder, F.Cu at (52.6, 56.5)
- added R67: 2.05k 1%, Resistor_SMD:R_0603_1608Metric_Pad0.98x0.95mm_HandSolder, F.Cu at (52.6, 59.0)
- added SW15: SW_Push, Button_Switch_SMD:SW_SPST_PTS645, F.Cu at (30.9, 33.4)
- added SW16: SW_Push, Button_Switch_SMD:SW_SPST_PTS645, F.Cu at (30.9, 41.3)
- added SW17: SW_Push, Button_Switch_SMD:SW_SPST_PTS645, F.Cu at (42.1, 17.7)
- added SW18: SW_Push, Button_Switch_SMD:SW_SPST_PTS645, F.Cu at (42.1, 25.6)
- added SW19: SW_Push, Button_Switch_SMD:SW_SPST_PTS645, F.Cu at (42.1, 33.4)
- added SW20: SW_Push, Button_Switch_SMD:SW_SPST_PTS645, F.Cu at (42.1, 41.3)
- added U11: USBLC6-2SC6, Package_TO_SOT_SMD:SOT-23-6, F.Cu at (-103.4, 63.5)
- added U12: TLV76133DCY, Package_TO_SOT_SMD:SOT-223-3_TabPin2, F.Cu at (-102.7, 54.9)
- added U8: 74HC14, Package_SO:SO-14_3.9x8.65mm_P1.27mm, F.Cu at (51.9, 19.1)
- added U9: 74HC14, Package_SO:SO-14_3.9x8.65mm_P1.27mm, F.Cu at (60.3, 19.1)
- C59, C60, C61, C62, C63, C64, D15, D16, D17, D18, D21, D22, D23, D24, D25, D26, R32, R33, R42, R43, R44, R45, R46, R47, R48, R49, R50, R51, R52, R53: moved to F.Cu
- R30: value 2.26k 1% -> 5.1k; footprint Resistor_SMD:R_0603_1608Metric_Pad0.98x0.95mm_HandSolder -> Resistor_SMD:R_0402_1005Metric; moved to F.Cu
- R31: value 2.05k 1% -> 5.1k; footprint Resistor_SMD:R_0603_1608Metric_Pad0.98x0.95mm_HandSolder -> Resistor_SMD:R_0402_1005Metric; moved to F.Cu
- moved SW5 176.0 mm to (-102.5, -7.80)
- moved D15 170.8 mm to (-88.2, -19.1), turned to 0 degrees
- moved D17 161.2 mm to (-82.4, -25.8), turned to 0 degrees
- moved SW7 158.4 mm to (-102.5, 7.90)
- moved C60 157.8 mm to (-94.0, -15.7), turned to 0 degrees
- moved C59 149.0 mm to (-94.0, -19.1), turned to 0 degrees
- moved D16 147.6 mm to (-88.2, -15.7), turned to 0 degrees
- moved SW4 147.1 mm to (-102.5, -15.7)
- moved R31 146.8 mm to (-104.5, 72.0), turned to 0 degrees
- moved SW6 146.1 mm to (-102.5, 0.05)
- moved R30 143.9 mm to (-104.5, 70.1)
- moved SW3 141.1 mm to (-102.5, -23.5)
- moved R43 139.2 mm to (-86.1, -5.24), turned to 0 degrees
- moved R42 139.1 mm to (-86.1, -7.75)
- moved R32 138.2 mm to (-94.8, -12.8)
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- renumbered C7 to C1, C16 to C10, C17 to C11, C18 to C12, C19 to C13, C20 to C14, C21 to C15, C22 to C16, C23 to C17, C24 to C18, C8 to C2, C25 to C20, C26 to C21, C27 to C23, C28 to C24, C29 to C25, C30 to C27, C31 to C29, C9 to C3, C32 to C30, C33 to C31, C34 to C32, C35 to C33, C36 to C34, C37 to C35, C38 to C36, C39 to C37, C40 to C38, C41 to C39, C10 to C4, C42 to C40, C43 to C41, C50 to C42, C51 to C43, C52 to C44, C53 to C45, C54 to C46, C55 to C47, C56 to C48, C57 to C49, C11 to C5, C58 to C50, C12 to C6, C13 to C7, C14 to C8, C15 to C9, D19 to D13, D20 to D14, D9 to D4, D4 to D5, D5 to D6, D6 to D7, D7 to D8, D8 to D9, FB2 to FB1, J3 to J2, J4 to J3, J1 to J4, J2 to J5, J5 to J6, R34 to R22, R35 to R23, R36 to R24, R37 to R25, R38 to R26, R39 to R27, R40 to R28, R41 to R29, U2 to U1, U3 to U2, U4 to U3, U5 to U4, U6 to U5, U8 to U6, U9 to U7
Connections:
- C59 pad 1: /Buttons/Debounced Button3/OUT_TO_SCHMIDT_TRIGGER -> (no net)
- C59 pad 2: GND -> (no net)
- C60 pad 1: /Buttons/Debounced Button4/OUT_TO_SCHMIDT_TRIGGER -> (no net)
- C60 pad 2: GND -> (no net)
- C61 pad 1: /Buttons/Debounced Button2/OUT_TO_SCHMIDT_TRIGGER -> (no net)
- C61 pad 2: GND -> (no net)
- C62 pad 1: /Buttons/Debounced Button5/OUT_TO_SCHMIDT_TRIGGER -> /Buttons/Debounced Button/OUT_TO_SCHMIDT_TRIGGER
- C63 pad 1: /Buttons/Debounced Button1/OUT_TO_SCHMIDT_TRIGGER -> /Keys/Debounced Button/OUT_TO_SCHMIDT_TRIGGER
- C64 pad 1: /Buttons/Debounced Button/OUT_TO_SCHMIDT_TRIGGER -> /Keys/Debounced Button7/OUT_TO_SCHMIDT_TRIGGER
- D15 pad 1: /Keys/Debounced Button2/OUT_TO_SCHMIDT_TRIGGER -> (no net)
- D15 pad 2: Net-(D15-A) -> (no net)
- D16 pad 1: /Keys/Debounced Button3/OUT_TO_SCHMIDT_TRIGGER -> (no net)
- D16 pad 2: Net-(D16-A) -> (no net)
- D17 pad 1: /Keys/Debounced Button4/OUT_TO_SCHMIDT_TRIGGER -> (no net)
- D17 pad 2: Net-(D17-A) -> (no net)
- D18 pad 1: /Keys/Debounced Button5/OUT_TO_SCHMIDT_TRIGGER -> (no net)
- D18 pad 2: Net-(D18-A) -> (no net)
- D21 pad 1: /Buttons/Debounced Button3/OUT_TO_SCHMIDT_TRIGGER -> /Keys/Debounced Button/OUT_TO_SCHMIDT_TRIGGER
- D21 pad 2: Net-(D21-A) -> Net-(D21-A)_1
- D22 pad 1: /Buttons/Debounced Button4/OUT_TO_SCHMIDT_TRIGGER -> /Keys/Debounced Button7/OUT_TO_SCHMIDT_TRIGGER
- D23 pad 1: /Buttons/Debounced Button2/OUT_TO_SCHMIDT_TRIGGER -> /Keys/Debounced Button1/OUT_TO_SCHMIDT_TRIGGER
- D24 pad 1: /Buttons/Debounced Button5/OUT_TO_SCHMIDT_TRIGGER -> /Keys/Debounced Button8/OUT_TO_SCHMIDT_TRIGGER
- D25 pad 1: /Buttons/Debounced Button1/OUT_TO_SCHMIDT_TRIGGER -> /Keys/Debounced Button2/OUT_TO_SCHMIDT_TRIGGER
- D26 pad 1: /Buttons/Debounced Button/OUT_TO_SCHMIDT_TRIGGER -> /Keys/Debounced Button3/OUT_TO_SCHMIDT_TRIGGER
- J2 pad 1: unconnected-(J3-Pin_1-Pad1) -> /AUDIO_INPUT_R
- J2 pad 2: unconnected-(J3-Pin_2-Pad2) -> GND
- J2 pad 3: unconnected-(J3-Pin_3-Pad3) -> /AUDIO_INPUT_L
- J3 pad 1: unconnected-(J4-Pin_1-Pad1) -> /BUFFERED_AUDIO_OUTPUT_L
- J3 pad 2: unconnected-(J4-Pin_2-Pad2) -> GND
- J3 pad 3: unconnected-(J4-Pin_3-Pad3) -> /BUFFERED_AUDIO_OUTPUT_R
- R30 pad 1: VCC -> Net-(J7-CC1)
- R30 pad 2: Net-(D17-A) -> GND
- R31 pad 1: Net-(D17-A) -> Net-(J7-CC2)
- R31 pad 2: /Keys/Debounced Button4/OUT_TO_SCHMIDT_TRIGGER -> GND
- R32 pad 1: VCC -> (no net)
- R32 pad 2: Net-(D18-A) -> (no net)
- R33 pad 1: Net-(D18-A) -> (no net)
- R33 pad 2: /Keys/Debounced Button5/OUT_TO_SCHMIDT_TRIGGER -> (no net)
- R43 pad 2: /Buttons/Debounced Button3/OUT_TO_SCHMIDT_TRIGGER -> /Buttons/Debounced Button/OUT_TO_SCHMIDT_TRIGGER
- R44 pad 2: Net-(D22-A) -> Net-(D21-A)_1
- R45 pad 1: Net-(D22-A) -> Net-(D21-A)_1
- R45 pad 2: /Buttons/Debounced Button4/OUT_TO_SCHMIDT_TRIGGER -> /Keys/Debounced Button/OUT_TO_SCHMIDT_TRIGGER
- R46 pad 2: Net-(D23-A) -> Net-(D22-A)
- R47 pad 1: Net-(D23-A) -> Net-(D22-A)
- R47 pad 2: /Buttons/Debounced Button2/OUT_TO_SCHMIDT_TRIGGER -> /Keys/Debounced Button7/OUT_TO_SCHMIDT_TRIGGER
- R48 pad 2: Net-(D24-A) -> Net-(D23-A)
- R49 pad 1: Net-(D24-A) -> Net-(D23-A)
- R49 pad 2: /Buttons/Debounced Button5/OUT_TO_SCHMIDT_TRIGGER -> /Keys/Debounced Button1/OUT_TO_SCHMIDT_TRIGGER
- R50 pad 2: Net-(D25-A) -> Net-(D24-A)
- R51 pad 1: Net-(D25-A) -> Net-(D24-A)
- R51 pad 2: /Buttons/Debounced Button1/OUT_TO_SCHMIDT_TRIGGER -> /Keys/Debounced Button8/OUT_TO_SCHMIDT_TRIGGER
- R52 pad 2: Net-(D26-A) -> Net-(D25-A)
- R53 pad 1: Net-(D26-A) -> Net-(D25-A)
- R53 pad 2: /Buttons/Debounced Button/OUT_TO_SCHMIDT_TRIGGER -> /Keys/Debounced Button2/OUT_TO_SCHMIDT_TRIGGER
- SW3 pad 1: Net-(D13-A) (its old number) -> (no net)
- SW3 pad 2: GND -> (no net)
- SW4 pad 1: Net-(D14-A) -> (no net)
- SW4 pad 2: GND -> (no net)
- SW5 pad 1: Net-(D15-A) -> (no net)
- SW5 pad 2: GND -> (no net)
- SW6 pad 1: Net-(D16-A) -> (no net)
- SW6 pad 2: GND -> (no net)
- SW7 pad 1: Net-(D17-A) -> (no net)
- SW7 pad 2: GND -> (no net)
- SW8 pad 1: Net-(D18-A) -> Net-(D21-A)
- SW9 pad 1: Net-(D21-A) -> Net-(D21-A)_1
Routing:
- net GND: track 158.4 -> 0.00 mm, vias 12 -> 11
- net Net-(D24-A): track 14.4 -> 0.00 mm
- net Net-(D26-A): track 14.4 -> 0.00 mm
- net Net-(D25-A): track 14.4 -> 0.00 mm
- net Net-(D21-A): track 14.4 -> 0.00 mm
- net Net-(D23-A): track 14.4 -> 0.00 mm
- net Net-(D18-A): track 14.4 -> 0.00 mm, vias 1 -> 0
- net Net-(D22-A): track 14.4 -> 0.00 mm
- net Net-(D15-A): track 14.4 -> 0.00 mm, vias 1 -> 0
- net Net-(D17-A): track 14.4 -> 0.00 mm, vias 1 -> 0
- net Net-(D16-A): track 14.4 -> 0.00 mm, vias 1 -> 0
- net Net-(D14-A): track 14.4 -> 0.00 mm, vias 1 -> 0
- net Net-(D13-A) (its old number): track 14.4 -> 0.00 mm, vias 1 -> 0
- net /Keys/Debounced Button2/OUT_TO_SCHMIDT_TRIGGER: track 5.42 -> 0.00 mm
- net /Buttons/Debounced Button3/OUT_TO_SCHMIDT_TRIGGER: track 5.42 -> 0.00 mm
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