File: pcb/BananaGuard.kicad_sch (KiCad schematic)
At the start: 16 parts, among them J1 AudioJack3_Ground, J2 AudioJack3_Ground, P1 USB_C_Plug_USB2.0, U1 TLV320AIC32IRHBR, U3 AMS1117-3.3

Commit message: ⚙️ wip, stm32 reference schem + jobset
Other:
- note added: "TODO: - dc jac/usb power - i2s connection with codec - pin defs (check cube mx to see what can be used where) - debug leds/other breakouts - 1x ws2812 for the guards staff - i2c for an oled or something possibly. - reinvestigate rp2040 (because the st dev environment is pain) - power filtering - analogue front/back end (preamp/buffering)"
- note added: "https://www.youtube.com/watch?v=zlGSxZGwj-E"
Changed lines of the file:
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@@
 (kicad_sch
-	(version 20231120)
+	(version 20250114)
 	(generator "eeschema")
-	(generator_version "8.0")
+	(generator_version "9.0")
 	(paper "A4")
+	(text "TODO:\n- dc jac/usb power \n- i2s connection with codec\n- pin defs (check cube mx to see what can be used where)\n- debug leds/other breakouts\n- 1x ws2812 for the guards staff\n- i2c for an oled or something possibly.\n- reinvestigate rp2040 (because the st dev environment is pain)\n- power filtering\n- analogue front/back end (preamp/buffering)"
+		(exclude_from_sim no)
+		(at 187.96 68.58 0)
+		(effects
+			(font
+				(size 1.27 1.27)
+			)
+			(justify left)
+		)
+	)
+	(text "https://www.youtube.com/watch?v=zlGSxZGwj-E"
+		(exclude_from_sim no)
+		(at 261.62 29.21 0)
+		(effects
+			(font
+				(size 5.08 5.08)
+			)
+		)
+	)
 	(junction
 		(at 48.26 74.93)
@@
 		(at 209.55 97.79)
 		(size 55.88 40.64)
+		(exclude_from_sim no)
+		(in_bom yes)
+		(on_board yes)
+		(dnp no)
 		(fields_autoplaced yes)
 		(stroke
@@
 		)
 		(instances
-			(project "BanannaFuzz"
+			(project "BananaGuard"
 				(path "/c334e595-b478-4c47-9288-968ac2c472fc"
 					(page "2")
@@
 		)
 	)
+	(embedded_fonts no)
 )

Commit message: 🎛  wip analogue front end
Parts:
- removed J1, J2: AudioJack3_Ground, Connector_Audio:Jack_3.5mm_PJ320E_Horizontal, symbol Connector_Audio:AudioJack3_Ground
- removed U3: AMS1117-3.3, Package_TO_SOT_SMD:SOT-223-3_TabPin2, symbol Regulator_Linear:AMS1117-3.3
- added C19, C21, C23, C25, C28: 0.1u, Capacitor_SMD:C_0603_1608Metric, symbol Device:C_Polarized
- added C20, C22, C24, C26, C29: 1u, Capacitor_SMD:CP_Elec_4x3, symbol Device:C_Polarized
- added C27: 10u, Capacitor_SMD:CP_Elec_4x3, symbol Device:C_Polarized
- added C4: 1u, Capacitor_SMD:CP_Elec_4x3, symbol Device:C
- added C7: 2.2u, Capacitor_SMD:CP_Elec_4x3, symbol Device:C
- added D5: WS2812, LED_SMD:LED_WS2812_PLCC6_5.0x5.0mm_P1.6mm, symbol LED:WS2812
- added D6, D7: LED, LED_SMD:LED_0603_1608Metric_Pad1.05x0.95mm_HandSolder, symbol Device:LED
- added J4, J5: Conn_01x04_Pin, Connector_PinHeader_2.54mm:PinHeader_1x04_P2.54mm_Vertical, symbol Connector:Conn_01x04_Pin
- added J6, J7: Conn_01x03_Socket, symbol Connector:Conn_01x03_Socket
- added R10, R11: 270, Resistor_SMD:R_0603_1608Metric_Pad0.98x0.95mm_HandSolder, symbol Device:R
- added R8, R9: 1k, Resistor_SMD:R_0603_1608Metric_Pad0.98x0.95mm_HandSolder, symbol Device:R
- added RV2, RV3, RV4: 10k, Potentiometer_THT:Potentiometer_Bourns_PTV09A-1_Single_Vertical, symbol Device:R_Potentiometer
- added U3: TLV76133DCY, Package_TO_SOT_SMD:SOT-223-3_TabPin2, symbol Regulator_Linear:TLV76133DCY
- RV1: value R_Potentiometer -> 10k; footprint (none) -> Potentiometer_THT:Potentiometer_Bourns_PTV09A-1_Single_Vertical
Connections:
- net +3.3V: now also RV1.1, U1.7 (IOVDD), C21.1, C22.1, C7.1, D5.3 (VCC), J4.4 (Pin_4), J5.4 (Pin_4), R8.1, R9.1, RV2.1, RV3.1, RV4.1, U3.2 (VO)
- net GND: now also D4.1 (K), U1.17 (AVSS1), U1.21 (DRVSS), U1.26 (AVSS2), U1.33 (EPAD), U1.6 (DVSS), C19.2, C20.2, C21.2, C22.2, C23.2, C24.2, C25.2, C26.2, C27.2, C28.2, C29.2, C4.2, C7.2, D5.6 (VSS), D6.1 (K), D7.1 (K), J4.1 (Pin_1), J5.1 (Pin_1), RV2.3, RV3.3, RV4.3, U3.1 (GND)
- net at R4.2: now also D4.2 (A)
- net POT1: now reaches RV1.2
- net USB_D+: now reaches P1.A6 (D+)
- net USB_D-: now reaches P1.A7 (D-)
- net I2S_MCK: now reaches U1.1 (MCLK)
- net +3.3VA: now reaches U1.18 (DRVDD)
- net +3.3VA: now also U1.24 (DRVDD), U1.25 (AVDD), C23.1, C24.1, C25.1, C26.1, C27.1, C28.1, C29.1
- net I2S_BCK: now reaches U1.2 (BCLK)
- net I2S_WS: now reaches U1.3 (WCLK)
- net ~{CODEC_RESET}: now reaches U1.31 (~{RESET})
- net +1.8V: now reaches U1.32 (DVDD)
- net +1.8V: now also C19.1, C20.1
- net I2S_SD_DAC: now reaches U1.4 (DIN)
- net I2S_SD_ADC: now reaches U1.5 (DOUT)
- net SCL: now reaches U1.8 (SCL)
- net SCL: now also J5.3 (Pin_3), R8.2
- net SDA: now reaches U1.9 (SDA)
- net SDA: now also J5.2 (Pin_2), R9.2
- removed net +5V: P1.A4 (VBUS), P1.A9 (VBUS), P1.B4 (VBUS), P1.B9 (VBUS), R1.1, R2.1, R3.1, R4.1, RV1.1
- new net: D7.2 (A), R11.2
- new net: D6.2 (A), R10.2
- new net DEBUG_LED1: R10.1
- new net DEBUG_LED2: R4.1
- new net DEBUG_LED3: R11.1
- new net HAT_LED1: R1.1
- new net HAT_LED2: R2.1
- new net HAT_LED3: R3.1
- new net LED_DIN: D5.2 (DIN)
- new net LED_DOUT: D5.1 (DOUT)
- new net POT2: RV2.2
- new net POT3: RV3.2
- new net POT4: RV4.2
- new net UART_RX: J4.2 (Pin_2)
- new net UART_TX: J4.3 (Pin_3)
- new net VBUS: C4.1, D5.5 (VDD), P1.A4 (VBUS), P1.A9 (VBUS), P1.B4 (VBUS), P1.B9 (VBUS), U3.3 (VI)
- no-connect marks 2 -> 3
Other:
- sheet MCU renamed STM32F429VIT6
- added sheet Analogue Front End (analogue.kicad_sch)
- sheet STM32F429VIT6 ports: added ADC1_IN0, ADC1_IN1, ADC1_IN2, ADC1_IN3, DAC_OUT1, DAC_OUT2, I2C1_SCL, I2C1_SDA, I2S2_CK, I2S2_EXT_SD, I2S2_SD, I2S2_WS, I2S_MCK, PA15, PA6, PA7, PA8, PB0, PB1, PB11, PB13, PB14, PB15, PB2, PB3, PB4, PB5, PB8, PB9, PC0, PC1, PC10, PC11, PC12, PC13, PC14, PC15, PC4, PC5, PC7, PC8, PC9, PD0, PD1, PD10, PD11, PD12, PD13, PD14, PD15, PD2, PD3, PD4, PD5, PD6, PD7, PD8, PD9, PE0, PE1, PE10, PE11, PE12, PE13, PE14, PE15, PE2, PE3, PE4, PE5, PE6, PE7, PE8, PE9, UART_RX, UART_TX, USB_D+, USB_D-; removed none
- note added: "I2S requires three pins, with an optional fourth pin: 1. Bit clock, using PB13 = I2S2_CK 2. Word clock, using PB12 = I2S2_WS 3. Serial data, using PB15 = I2S2_SD 4. Master clock, using PC6 = I2S2_MCK"
- note added: "TODO: - dc jac/usb power - i2s connection with codec - pin defs (check cube mx to see what can be used where) - debug leds/other breakouts - 1x ws2812 for the guards staff - i2c for an oled or something possibly. - reinvestigate rp2040 (because the st dev environment is pain) - power filtering - analogue front/back end (preamp/buffering) - usb protection circuitry"
- note added: "adc/dac"
- note added: "audio in (stereo) jst"
- note added: "audio out (stereo) jst"
- note added: "codec decoupling keep caps close to pins as labeled we are sharing gnd in this design."
- note added: "debug leds"
- note added: "expansion"
- note added: "hat gems"
- note added: "i2c breakout (oled or other peripherals)"
- note added: "io"
- note added: "mcu"
- note added: "power"
- note added: "staff led"
- note added: "uart breakout"
- note removed: "TODO: - dc jac/usb power - i2s connection with codec - pin defs (check cube mx to see what can be used where) - debug leds/other breakouts - 1x ws2812 for the guards staff - i2c for an oled or something possibly. - reinvestigate rp2040 (because the st dev environment is pain) - power filtering - analogue front/back end (preamp/buffering)"
- company: (none) -> kevontheweb
- title: (none) -> Banana Guard DSP
- moved on the sheet: D1, D2, D3, D4, H1, H2, P1, R1, R2, R3, R4, RV1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

Commit message: analogue fe +  buttons/keys
Parts:
- added C16, C18: 1u, Capacitor_SMD:CP_Elec_4x3, symbol Device:C_Polarized
- added C17: 100n, Capacitor_SMD:C_0603_1608Metric, symbol Device:C
- added C2: 10n, Capacitor_SMD:C_0603_1608Metric, symbol Device:C
- added C34: 47u, symbol Device:C
- added C35, C37, C38: 2.2u, Capacitor_SMD:C_0603_1608Metric, symbol Device:C
- added C39: 1u, Capacitor_SMD:C_0603_1608Metric, symbol Device:C
- added D10, D9: D_Schottky, symbol Device:D_Schottky
- added D18: WS2812, LED_SMD:LED_WS2812_PLCC6_5.0x5.0mm_P1.6mm, symbol LED:WS2812
- added FB1, FB2: 120R, Resistor_SMD:R_0603_1608Metric, symbol Device:FerriteBead
- added R16, R17: 1k, symbol Device:R
- added U7: TLV76150DCY, Package_TO_SOT_SMD:SOT-223-3_TabPin2, symbol Regulator_Linear:TLV76150DCY
Connections:
- net +3.3V: now also C18.1, C2.1, D18.3 (VCC), FB1.1
- net +3.3VA: now also C16.1, C17.1, FB1.2
- net GND: now also C16.2, C17.2, C18.2, C2.2, C35.2, C37.2, C38.2, C39.2, D18.6 (VSS), D9.2 (A), U7.1 (GND)
- net LED_DOUT: now also D18.1 (DOUT); no longer D5.1 (DOUT)
- net VBUS: now also D10.2 (A), D18.5 (VDD)
- net BUFFERED_AUDIO_INPUT_L: now reaches U1.10 (MIC1L/LINE1L)
- net BUFFERED_AUDIO_INPUT_R: now reaches U1.11 (MIC1R/LINE1R)
- net CODEC_AUDIO_OUTPUT_L: now reaches U1.27 (LEFT_LOP)
- net CODEC_AUDIO_OUTPUT_L_MINUS: now reaches U1.28 (LEFT_LOM)
- net CODEC_AUDIO_OUTPUT_R: now reaches U1.29 (RIGHT_LOP)
- net CODEC_AUDIO_OUTPUT_R_MINUS: now reaches U1.30 (RIGHT_LOM)
- new net: C37.1, C39.1, D10.1 (K), FB2.2, U7.3 (VI)
- new net: C34.2, R16.1
- new net: D18.2 (DIN), D5.1 (DOUT)
- new net +2.5V: C34.1, R16.2, R17.1
- new net +5V: C38.1, R17.2, U7.2 (VO)
- new net VCC: C35.1, D9.1 (K), FB2.1
- no-connect marks 3 -> 11
Other:
- added sheet Analogue Front End1 (analogue.kicad_sch)
- added sheet Buttons (keys.kicad_sch)
- added sheet Keys (keys.kicad_sch)
- sheet Analogue Front End ports: added AUDIO_INPUT, BUFFERED_AUDIO_INPUT, BUFFERED_AUDIO_OUTPUT, CODEC_AUDIO_OUTPUT; removed none
- note added: "0 dB = 0.707 V"
- note added: "?"
- note added: "analogue supply decoupling (common ground)"
- note added: "left"
- note added: "low esr (tantalum)"
- note added: "octave led"
- note added: "power for analogue front end"
- note added: "pwr in from dc jack/jst"
- note added: "pwr in from usb (ORing)"
- note added: "reference voltage"
- note added: "right"
- moved on the sheet: C19, C20, C21, C22, C23, C24, C25, C26, C27, C28, C29, C4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

Commit message: more schematic stuff, preliminary footprint choices and parts grouping, played with multicahnnel for the buttons
Parts:
- C11: renamed from C34; footprint (none) -> Capacitor_SMD:CP_Elec_4x3
- D10, D9: footprint (none) -> Diode_SMD:D_SOD-123
- J3: renamed from J6; footprint (none) -> Connector_JST:JST_ZE_B03B-ZESK-1D_1x03_P1.50mm_Vertical
- J4: renamed from J7; footprint (none) -> Connector_JST:JST_ZE_B03B-ZESK-1D_1x03_P1.50mm_Vertical
- R7: renamed from R17; footprint (none) -> Resistor_SMD:R_0603_1608Metric_Pad0.98x0.95mm_HandSolder
- R8: renamed from R16; footprint (none) -> Resistor_SMD:R_0603_1608Metric_Pad0.98x0.95mm_HandSolder
- renumbered C4 to C1, C38 to C10, C23 to C12, C19 to C13, C24 to C14, C20 to C15, C25 to C16, C21 to C17, C26 to C18, C22 to C19, C7 to C2, C27 to C20, C28 to C21, C29 to C22, C2 to C3, C18 to C4, C17 to C5, C16 to C6, C35 to C7, C37 to C8, C39 to C9, D6 to D1, D1 to D2, D5 to D3, D2 to D5, D18 to D6, D3 to D8, J4 to J1, J5 to J2, R10 to R1, R9 to R10, R1 to R2, R4 to R3, R2 to R4, R11 to R5, R3 to R6, R8 to R9, U3 to U1, U7 to U2, U1 to U3

Commit message: expand usb, piano keys, cleanup
Parts:
- removed C1: 1u, Capacitor_SMD:CP_Elec_4x3, symbol Device:C
- removed C2: 2.2u, Capacitor_SMD:CP_Elec_4x3, symbol Device:C
- removed C3: 10n, Capacitor_SMD:C_0603_1608Metric, symbol Device:C
- removed C4, C6: 1u, Capacitor_SMD:CP_Elec_4x3, symbol Device:C_Polarized
- removed C5: 100n, Capacitor_SMD:C_0603_1608Metric, symbol Device:C
- removed FB1: 120R, Resistor_SMD:R_0603_1608Metric, symbol Device:FerriteBead
- removed P1: USB_C_Plug_USB2.0, Connector_USB:USB_C_Receptacle_GCT_USB4105-xx-A_16P_TopMnt_Horizontal, symbol Connector:USB_C_Plug_USB2.0
- removed U1: TLV76133DCY, Package_TO_SOT_SMD:SOT-223-3_TabPin2, symbol Regulator_Linear:TLV76133DCY
- added J1: Conn_01x03_Socket, Connector_JST:JST_ZE_B03B-ZESK-1D_1x03_P1.50mm_Vertical, symbol Connector:Conn_01x03_Socket
- renumbered C7 to C1, C16 to C10, C17 to C11, C18 to C12, C19 to C13, C20 to C14, C21 to C15, C22 to C16, C8 to C2, C9 to C3, C10 to C4, C11 to C5, C12 to C6, C13 to C7, C14 to C8, C15 to C9, D9 to D4, D4 to D5, D5 to D6, D6 to D7, D7 to D8, D8 to D9, FB2 to FB1, J3 to J2, J4 to J3, J1 to J4, J2 to J5, U2 to U1, U3 to U2
Connections:
- net AUDIO_INPUT_L: now also J2.3 (Pin_3)
- net AUDIO_INPUT_R: now also J2.1 (Pin_1)
- net BUFFERED_AUDIO_OUTPUT_L: now also J3.1 (Pin_1)
- net BUFFERED_AUDIO_OUTPUT_R: now also J3.3 (Pin_3)
- net GND: now also J2.2 (Pin_2), J3.2 (Pin_2), J1.1 (Pin_1)
- net VCC: now also J1.3 (Pin_3)
- no-connect marks 11 -> 10
Other:
- sheet Analogue Front End renamed Analogue Front End Left
- sheet Analogue Front End1 renamed Analogue Front End Right
- added sheet USB (USB.kicad_sch)
- sheet Buttons: file keys.kicad_sch -> buttons.kicad_sch
- note added: "to DC barrel (JST)"
- note added: "usb/power"
- note removed: "analogue supply decoupling (common ground)"
- note removed: "power"
- moved on the sheet: C1, C10, C11, C12, C13, C14, C15, C16, C2, C3, C4, C5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

Commit message: switch back to rp2350, ideal diode OR'ing for power
Parts:
- removed D10, D4: D_Schottky, Diode_SMD:D_SOD-123, symbol Device:D_Schottky
- removed R10, R9: 1k, Resistor_SMD:R_0603_1608Metric_Pad0.98x0.95mm_HandSolder, symbol Device:R
- added C1: 10n, Capacitor_SMD:C_0603_1608Metric, symbol Device:C
- added C10, C75: 1u, Capacitor_SMD:CP_Elec_4x3, symbol Device:C
- added C11, C76: 2.2u, Capacitor_SMD:CP_Elec_4x3, symbol Device:C
- added C2, C4: 1u, Capacitor_SMD:CP_Elec_4x3, symbol Device:C_Polarized
- added C3: 100n, Capacitor_SMD:C_0603_1608Metric, symbol Device:C
- added C77, C78: 100n, Capacitor_SMD:CP_Elec_4x3, symbol Device:C
- added FB1: 120R, Resistor_SMD:R_0603_1608Metric, symbol Device:FerriteBead
- added R11: 20k, Resistor_SMD:R_0603_1608Metric_Pad0.98x0.95mm_HandSolder, symbol Device:R
- added R13: 10k, Resistor_SMD:R_0603_1608Metric_Pad0.98x0.95mm_HandSolder, symbol Device:R
- added R68, R69: 2k, Resistor_SMD:R_0603_1608Metric_Pad0.98x0.95mm_HandSolder, symbol Device:R
- added R70, R71, R72: 1k, Resistor_SMD:R_0603_1608Metric_Pad0.98x0.95mm_HandSolder, symbol Device:R
- added U13: TPS2116DRL, Package_TO_SOT_SMD:SOT-583-8, symbol Power_Management:TPS2116DRL
- added U14: TLV76718DRVx, Package_SON:WSON-6-1EP_2x2mm_P0.65mm_EP1x1.6mm_ThermalVias, symbol Regulator_Linear:TLV76718DRVx
- added U2: TLV76133DCY, Package_TO_SOT_SMD:SOT-223-3_TabPin2, symbol Regulator_Linear:TLV76133DCY
- renumbered C6 to C12, C7 to C13, C8 to C14, C9 to C15, C10 to C16, C11 to C17, C12 to C18, C13 to C19, C14 to C20, C15 to C21, C16 to C22, C1 to C5, C2 to C6, C3 to C7, C5 to C8, C4 to C9, D5 to D4, D6 to D5, FB1 to FB2, J4 to J2, J5 to J3, J2 to J4, J3 to J5, U2 to U3
Connections:
- net CODEC_AUDIO_OUTPUT_R_MINUS is gone; now on net CODEC_AUDIO_OUTPUT_MINUS_COM: U3.30 (RIGHT_LOM)
- net +1.8V: now also C76.1, U14.1 (OUT)
- net +3.3V: now also C1.1, C11.1, C2.1, C75.1, FB1.1, R70.1, R71.1, U14.4 (EN), U14.6 (IN), U2.2 (VO)
- net +3.3VA: now also C3.1, C4.1, FB1.2
- net +5V: now also C10.1, U2.3 (VI)
- net BUFFERED_AUDIO_INPUT_L: now also C77.1; no longer U3.10 (MIC1L/LINE1L)
- net BUFFERED_AUDIO_INPUT_R: now also C78.1; no longer U3.11 (MIC1R/LINE1R)
- net GND: now also C1.2, C10.2, C11.2, C2.2, C3.2, C4.2, C75.2, C76.2, R13.1, U13.1 (GND), U14.3 (GND), U14.5 (GND), U14.7 (PAD), U2.1 (GND); no longer J5.2 (Pin_2)
- net SCL: now also R71.2
- net SDA: now also R70.2
- net VBUS: now also R11.2, R72.1, U13.3 (VIN1), U13.5 (MODE)
- net VCC: now also U13.6 (VIN2); no longer C5.1, FB2.1
- net at U3.15 (MICBIAS): now also R68.1, R69.1
- net CODEC_AUDIO_OUTPUT_L_MINUS renamed CODEC_AUDIO_OUTPUT_MINUS_COM
- net CODEC_AUDIO_OUTPUT_MINUS_COM: now also J5.2 (Pin_2)
- new net: C5.1, FB2.1, U13.2 (VOUT), U13.7 (VOUT)
- new net: R11.1, R13.2, U13.4 (PR1)
- new net: R72.2, U13.8 (ST)
- new net: C78.2, R68.2, U3.11 (MIC1R/LINE1R)
- new net: C77.2, R69.2, U3.10 (MIC1L/LINE1L)
Other:
- removed sheet STM32F429VIT6
- added sheet RP2350B (RP2350B.kicad_sch)
- note added: "Power"
- note added: "analogue supply decoupling (common ground) (probably not necessary since we are already using a ferrite bead before 5v out and the 5v is being used to power the op amps anyway)"
- note added: "gnd?"
- note added: "jst header to panel mount DC barrel jack"
- note added: "low esr x5r"
- note added: "reference voltage for opamps"
- note added: "usb"
- note added: "vout=vfb*(1+r1/r2)"
- note added: "will prefer vin1 but switch to vin2 when vin1 is less than 2V, to switch back vin1 must be greater than 3V if either are less than 1.6 vout is hiZ"
- note removed: "?"
- note removed: "low esr (tantalum)"
- note removed: "power for analogue front end"
- note removed: "reference voltage"
- note removed: "to DC barrel (JST)"
- note removed: "usb/power"
- moved on the sheet: C12, C13, C14, C15, C16, C17, C18, C19, C20, C21, C22, C5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
