File: pcb/buttons.kicad_sch (KiCad schematic)
At the start: 1 part, among them U10 74HC14

Commit message: switch back to rp2350, ideal diode OR'ing for power
Parts:
- renumbered U10 to U11
Changed lines of the file:
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@@
 		(dnp no)
 		(fields_autoplaced yes)
-		(property "Reference" "U10"
+		(property "Reference" "U11"
 			(at 41.91 45.7199 0)
 			(effects
@@
 				)
 				(path "/c334e595-b478-4c47-9288-968ac2c472fc/ae7f9a36-3daf-4903-87c4-e09344dfdb56"
-					(reference "U10")
+					(reference "U11")
 					(unit 7)
 				)
@@
 		(dnp no)
 		(fields_autoplaced yes)
-		(property "Reference" "#PWR099"
+		(property "Reference" "#PWR0143"
 			(at 35.56 66.04 0)
 			(effects
@@
 			(project "BananaGuard"
 				(path "/c334e595-b478-4c47-9288-968ac2c472fc/ae7f9a36-3daf-4903-87c4-e09344dfdb56"
-					(reference "#PWR099")
+					(reference "#PWR0143")
 					(unit 1)
 				)
@@
 		(dnp no)
 		(fields_autoplaced yes)
-		(property "Reference" "U10"
+		(property "Reference" "U11"
 			(at 110.49 80.01 0)
 			(effects
@@
 				)
 				(path "/c334e595-b478-4c47-9288-968ac2c472fc/ae7f9a36-3daf-4903-87c4-e09344dfdb56"
-					(reference "U10")
+					(reference "U11")
 					(unit 3)
 				)
@@
 		(dnp no)
 		(fields_autoplaced yes)
-		(property "Reference" "U10"
+		(property "Reference" "U11"
 			(at 110.49 156.21 0)
 			(effects
@@
 				)
 				(path "/c334e595-b478-4c47-9288-968ac2c472fc/ae7f9a36-3daf-4903-87c4-e09344dfdb56"
-					(reference "U10")
+					(reference "U11")
 					(unit 6)
 				)
@@
 		(dnp no)
 		(fields_autoplaced yes)
-		(property "Reference" "U10"
+		(property "Reference" "U11"
 			(at 110.49 130.81 0)
 			(effects
@@
 				)
 				(path "/c334e595-b478-4c47-9288-968ac2c472fc/ae7f9a36-3daf-4903-87c4-e09344dfdb56"
-					(reference "U10")
+					(reference "U11")
 					(unit 5)
 				)
@@
 		(dnp no)
 		(fields_autoplaced yes)
-		(property "Reference" "#PWR098"
+		(property "Reference" "#PWR0142"
 			(at 35.56 38.1 0)
 			(effects
@@
 			(project "BananaGuard"
 				(path "/c334e595-b478-4c47-9288-968ac2c472fc/ae7f9a36-3daf-4903-87c4-e09344dfdb56"
-					(reference "#PWR098")
+					(reference "#PWR0142")
 					(unit 1)
 				)
@@
 		(dnp no)
 		(fields_autoplaced yes)
-		(property "Reference" "U10"
+		(property "Reference" "U11"
 			(at 110.49 105.41 0)
 			(effects
@@
 				)
 				(path "/c334e595-b478-4c47-9288-968ac2c472fc/ae7f9a36-3daf-4903-87c4-e09344dfdb56"
-					(reference "U10")
+					(reference "U11")
 					(unit 4)
 				)
@@
 		(dnp no)
 		(fields_autoplaced yes)
-		(property "Reference" "U10"
+		(property "Reference" "U11"
 			(at 110.49 54.61 0)
 			(effects
@@
 				)
 				(path "/c334e595-b478-4c47-9288-968ac2c472fc/ae7f9a36-3daf-4903-87c4-e09344dfdb56"
-					(reference "U10")
+					(reference "U11")
 					(unit 2)
 				)
@@
 		(dnp no)
 		(fields_autoplaced yes)
-		(property "Reference" "U10"
+		(property "Reference" "U11"
 			(at 110.49 29.21 0)
 			(effects
@@
 				)
 				(path "/c334e595-b478-4c47-9288-968ac2c472fc/ae7f9a36-3daf-4903-87c4-e09344dfdb56"
-					(reference "U10")
+					(reference "U11")
 					(unit 1)
 				)
